Commit message: Updated models

File: src/myrobot/models/structure.urdf (robot description, URDF)
Before this commit: robot structure, 3 links, 2 joints
Links:
- removed link link
- added link main_base, mass 1; collision cylinder length=3 radius=1; visual box size=0.15 4 0.15
- added link side_one, mass 1; collision cylinder length=3 radius=1; visual box size=0.15 0.15 3
- added link side_two, mass 1; collision cylinder length=3 radius=1; visual box size=0.15 0.15 3
Joints:
- added joint sideconn1: type fixed, parent main_base, child side_one, origin xyz=0 0 0
- added joint sideconn2: type fixed, parent main_base, child side_two, origin xyz=0 0 0
- joint boxconnect1: parent link -> main_base
- joint boxconnect2: parent link -> main_base

Commit message: COmpleted static structure

File: src/myrobot/models/structure.urdf (robot description, URDF)
Before this commit: robot structure, 5 links, 4 joints
Links:
- link main_base: geometry collision box size=0.15 4 0.15; visual box size=0.15 4 0.15
- link side_one: geometry collision box size=0.15 0.15 3; visual box size=0.15 0.15 3
- link side_two: geometry collision box size=0.15 0.15 3; visual box size=0.15 0.15 3
