Commit message: Updated something

File: src/myrobot/models/forklift.urdf (robot description, URDF)
Before this commit: robot forklift, 1 links, 0 joints
Links:
- removed link forklift_base
- added link back_wheel, mass 0.114; collision mesh filename=package://myrobot/models/forklift/meshes/forklift_back_whee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 scale=0.01 0.01 0.01; visual mesh filename=package://myrobot/models/forklift/meshes/forklift_back_whee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 scale=0.01 0.01 0.01
- added link forklift_chassis, mass 0.114; collision mesh filename=package://myrobot/models/forklift/meshes/forklift_chassis.s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 scale=0.01 0.01 0.01; visual mesh filename=package://myrobot/models/forklift/meshes/forklift_chassis.s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 scale=0.01 0.01 0.01
- added link left_wheel, mass 0.114; collision mesh filename=package://myrobot/models/forklift/meshes/forklift_left_whee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 scale=0.01 0.01 0.01; visual mesh filename=package://myrobot/models/forklift/meshes/forklift_left_whee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 scale=0.01 0.01 0.01
- added link right_wheel, mass 0.114; collision mesh filename=package://myrobot/models/forklift/meshes/forklift_right_whe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 scale=0.01 0.01 0.01; visual mesh filename=package://myrobot/models/forklift/meshes/forklift_right_whe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 scale=0.01 0.01 0.01
Joints:
- added joint back_wheel_joint: type continuous, parent forklift_chassis, child back_wheel, origin xyz=0 0 0, axis 1 0 0
- added joint left_wheel_joint: type continuous, parent forklift_chassis, child left_wheel, origin xyz=0 0 0, axis 1 0 0
- added joint right_wheel_joint: type continuous, parent forklift_chassis, child right_wheel, origin xyz=0 0 0, axis 1 0 0
